Commit message: Updated launch files for successful rviz launch

File: scout/scout_description/urdf/scout_mini.xacro (robot description, xacro)
@@ -15,6 +15,6 @@
     <xacro:property name="base_z_size" value="0.235000" />
     <xacro:property name="wheelbase" value="0.3132556"/>
-   <xacro:property name="track" value="0.4563536" />
-   <xacro:property name="wheel_vertical_offset" value="-0.077" />
+    <xacro:property name="track" value="0.4563536" />
+    <xacro:property name="wheel_vertical_offset" value="-0.077" />
 <!--    <xacro:property name="track" value="0.3426" />
     <xacro:property name="wheelbase" value="0.3181"/>

Commit message: Updated xacro and launch files for gazebo compatability

File: scout/scout_description/urdf/scout_mini.xacro (robot description, xacro)
@@ -4,4 +4,5 @@
     <xacro:arg name="robot_namespace" default="/" />
     <xacro:arg name="urdf_extras" default="empty.urdf" />
+    <!-- Include wheel definitions -->
     <xacro:include filename="$(find scout_description)/urdf/scout_mini_wheel_1.xacro" />
     <xacro:include filename="$(find scout_description)/urdf/scout_mini_wheel_2.xacro" />
@@ -9,25 +10,20 @@
     <xacro:include filename="$(find scout_description)/urdf/scout_mini_wheel_4.xacro" />
     <!-- Variables -->
-    <xacro:property name="M_PI" value="3.14159"/>
+    <xacro:property name="M_PI" value="3.14159" />
     <!-- Vehicle Geometries -->
     <xacro:property name="base_x_size" value="0.6200000" />
     <xacro:property name="base_y_size" value="0.585000" />
     <xacro:property name="base_z_size" value="0.235000" />
-    <xacro:property name="wheelbase" value="0.3132556"/>
+    <xacro:property name="wheelbase" value="0.3132556" />
     <xacro:property name="track" value="0.4563536" />
     <xacro:property name="wheel_vertical_offset" value="-0.077" />
-<!--    <xacro:property name="track" value="0.3426" />
-    <xacro:property name="wheelbase" value="0.3181"/>
-    <xacro:property name="wheel_vertical_offset" value="-0.160000047342231" />-->
     <xacro:property name="wheel_length" value="0.8e-01" />
     <xacro:property name="wheel_radius" value="1.600e-01" />
+    <!-- For easier debugging, define base_z_offset -->
+    <xacro:property name="base_z_offset" value="${base_z_size / 2}" />
     <!-- Base link -->
     <link name="base_link">
         <visual>
-            <!--origin xyz="-0.0145261552504705 0.0231316650320557 0.00586280190939592" rpy="0 0 0" /-->
             <origin xyz="0.015 0.0231316650320557 0" rpy="0 0 0"/>
-            <!--<origin
-              xyz="-0.0145261552504705 0.0231316650320557 0.00586280190939592"
-              rpy="0 0 0" />-->
             <geometry>
                 <mesh filename="package://scout_description/meshes/scout_mini_base_link.STL" />
@@ -35,39 +31,23 @@
         </visual>
         <collision>
-          <!--origin
-            xyz="-0.0145261552504705 0.0231316650320557 0.00586280190939592"
-            rpy="0 0 0" /-->
-            <origin xyz="0.015 0.0231316650320557 0" rpy="0 0 0"/>
-          <geometry>
-            <mesh
-              filename="package://scout_description/meshes/scout_mini_base_link.STL" />
-          </geometry>
+            <geometry>
+                <box size="${base_x_size} ${base_y_size} ${base_z_size}" />
+            </geometry>
         </collision>
     </link>
-    <!-- <joint name="chassis_link_joint" type="fixed">
-        <origin xyz="0 0 ${wheel_radius - wheel_vertical_offset}" rpy="0 0 0" />
-        <parent link="base_link" />
-        <child link="chassis_link" />
-    </joint> -->
+    <!-- Inertial link -->
     <link name="inertial_link">
         <inertial>
-            <!--mass value="44.3898489950015" /-->
             <mass value="132.3898489950015" />
-            <!-- <mass value="50" /> -->
-            <!-- <origin xyz="-0.00065 -0.085 0.062" />
-            <inertia ixx="0.6022" ixy="-0.02364" ixz="-0.1197" iyy="1.7386" iyz="-0.001544" izz="2.0296" /> -->
-            <origin xyz="0.015 0.0231316650320557 0" />
-            <!--<origin
-              xyz="-0.0145261552504705 0.0231316650320557 0.00586280190939592"
-              rpy="0 0 0" />-->
+            <origin xyz="0 0 ${base_z_offset}" />
             <inertia ixx="0.185196122711036"
-            ixy="4.30144213829512E-08"
-            ixz="5.81037523686401E-08"
-            iyy="0.364893736238929"
-            iyz="-0.000386720198091934"
-            izz="0.223868521722778" />
-            <!--<inertia ixx="2.288641" ixy="0" ixz="0" iyy="5.103976" iyz="0" izz="3.431465" />-->
+                     ixy="4.30144213829512E-08"
+                     ixz="5.81037523686401E-08"
+                     iyy="0.364893736238929"
+                     iyz="-0.000386720198091934"
+                     izz="0.223868521722778" />
         </inertial>
     </link>
+    <!-- Inertial joint -->
     <joint name="inertial_joint" type="fixed">
         <origin xyz="0 0 0" rpy="0 0 0" />
@@ -75,25 +55,18 @@
         <child link="inertial_link" />
     </joint>
-    <!-- For testing, hang the robot up in the air -->
-    <!-- <link name="world" />
-    <joint name="world_to_base_link=" type="fixed">
-        <origin xyz="0 0 0.5" rpy="0 0 0" />
-        <parent link="world"/>
-        <child link="base_link"/>
-    </joint> -->
     <!-- Scout wheel macros -->
-    <!-- wheel labeled from 0 to 3, conter-clockwise, starting from front right wheel -->
+    <!-- wheel labeled from 0 to 3, counter-clockwise, starting from front right wheel -->
     <!-- motor 1 and 2 (left side) are mechanically installed in a reversed direction -->
     <xacro:scout_mini_wheel_1 wheel_prefix="rear_right">
-        <origin xyz="${wheelbase/2} ${-track/2} ${wheel_vertical_offset}" rpy="0 1.57 0" />
+        <origin xyz="${wheelbase / 2} ${-track / 2} ${wheel_vertical_offset}" rpy="0 1.57 0" />
     </xacro:scout_mini_wheel_1>
     <xacro:scout_mini_wheel_2 wheel_prefix="front_right">
-        <origin xyz="${wheelbase/2} ${track/2} ${wheel_vertical_offset}" rpy="0 1.57 0" />
+        <origin xyz="${wheelbase / 2} ${track / 2} ${wheel_vertical_offset}" rpy="0 1.57 0" />
     </xacro:scout_mini_wheel_2>
     <xacro:scout_mini_wheel_3 wheel_prefix="front_left">
-        <origin xyz="${-wheelbase/2} ${track/2} ${wheel_vertical_offset}" rpy="0 -1.57 0" />
+        <origin xyz="${-wheelbase / 2} ${track / 2} ${wheel_vertical_offset}" rpy="0 -1.57 0" />
     </xacro:scout_mini_wheel_3>
     <xacro:scout_mini_wheel_4 wheel_prefix="rear_left">
-        <origin xyz="${-wheelbase/2} ${-track/2} ${wheel_vertical_offset}" rpy="0 -1.57 0" />
+        <origin xyz="${-wheelbase / 2} ${-track / 2} ${wheel_vertical_offset}" rpy="0 -1.57 0" />
     </xacro:scout_mini_wheel_4>
     <!-- Additional definitions -->

Commit message: Updated xacro files for robot base visibility in Gazebo

File: scout/scout_description/urdf/scout_mini.xacro (robot description, xacro)
@@ -12,7 +12,7 @@
     <xacro:property name="M_PI" value="3.14159" />
     <!-- Vehicle Geometries -->
-    <xacro:property name="base_x_size" value="0.6200000" />
-    <xacro:property name="base_y_size" value="0.585000" />
-    <xacro:property name="base_z_size" value="0.235000" />
+    <!-- xacro:property name="base_x_size" value="0.6200000" /-->
+    <!-- xacro:property name="base_y_size" value="0.585000" /-->
+    <!-- xacro:property name="base_z_size" value="0.235000" /-->
     <xacro:property name="wheelbase" value="0.3132556" />
     <xacro:property name="track" value="0.4563536" />
@@ -20,19 +20,26 @@
     <xacro:property name="wheel_length" value="0.8e-01" />
     <xacro:property name="wheel_radius" value="1.600e-01" />
-    <!-- For easier debugging, define base_z_offset -->
-    <xacro:property name="base_z_offset" value="${base_z_size / 2}" />
+    <!-- xacro:property name="base_z_offset" value="0.5" /-->
     <!-- Base link -->
     <link name="base_link">
+        <inertial>
+            <mass value="10" />
+            <origin xyz="0 0 0.5" />
+            <inertia ixx="0.1" ixy="0.0" ixz="0.0" iyy="0.1" iyz="0.0" izz="0.1" />
+        </inertial>
         <visual>
             <origin xyz="0.015 0.0231316650320557 0" rpy="0 0 0"/>
             <geometry>
-                <mesh filename="package://scout_description/meshes/scout_mini_base_link.STL" />
+                <mesh filename="package://scout_description/meshes/scout_mini_base_link.STL"/>
             </geometry>
         </visual>
         <collision>
             <geometry>
-                <box size="${base_x_size} ${base_y_size} ${base_z_size}" />
+                <box size="0.6200000 0.585000 0.235000" />
             </geometry>
         </collision>
+        <gazebo>
+            <material>Gazebo/Blue</material>
+        </gazebo>
     </link>
     <!-- Inertial link -->
@@ -40,5 +47,5 @@
         <inertial>
             <mass value="132.3898489950015" />
-            <origin xyz="0 0 ${base_z_offset}" />
+            <origin xyz="0 0 0.5" />
             <inertia ixx="0.185196122711036"
                      ixy="4.30144213829512E-08"
@@ -48,4 +55,5 @@
                      izz="0.223868521722778" />
         </inertial>
+        <gazebo/>
     </link>
     <!-- Inertial joint -->
