Commit message: Add lidar sensor

File: scout/scout_description/urdf/scout_mini.xacro (robot description, xacro)
@@ -1,7 +1,7 @@
 <?xml version="1.0"?>
 <robot name="scout_mini"
-    xmlns:xacro="http://ros.org/wiki/xacro">
+       xmlns:xacro="http://ros.org/wiki/xacro">
     <xacro:arg name="robot_namespace" default="/" />
-    <xacro:arg name="urdf_extras" default="empty.urdf" />
+    <xacro:arg name="urdf_extras" default="$(find scout_description)/urdf/empty.urdf" />
     <!-- Include wheel definitions -->
     <xacro:include filename="$(find scout_description)/urdf/scout_mini_wheel_1.xacro" />
@@ -9,16 +9,4 @@
     <xacro:include filename="$(find scout_description)/urdf/scout_mini_wheel_3.xacro" />
     <xacro:include filename="$(find scout_description)/urdf/scout_mini_wheel_4.xacro" />
-    <!-- Variables -->
-    <xacro:property name="M_PI" value="3.14159" />
-    <!-- Vehicle Geometries -->
-    <!-- xacro:property name="base_x_size" value="0.6200000" /-->
-    <!-- xacro:property name="base_y_size" value="0.585000" /-->
-    <!-- xacro:property name="base_z_size" value="0.235000" /-->
-    <xacro:property name="wheelbase" value="0.3132556" />
-    <xacro:property name="track" value="0.4563536" />
-    <xacro:property name="wheel_vertical_offset" value="-0.077" />
-    <xacro:property name="wheel_length" value="0.8e-01" />
-    <xacro:property name="wheel_radius" value="1.600e-01" />
-    <!-- xacro:property name="base_z_offset" value="0.5" /-->
     <!-- Base link -->
     <link name="base_link">
@@ -29,12 +17,12 @@
         </inertial>
         <visual>
-            <origin xyz="0.015 0.0231316650320557 0" rpy="0 0 0"/>
+            <origin xyz="0.015 0.023 0" rpy="0 0 0"/>
             <geometry>
-                <mesh filename="package://scout_description/meshes/scout_mini_base_link.STL"/>
+                <mesh filename="package://scout_description/meshes/scout_mini_base_link.STL" scale="1 1 1" />
             </geometry>
         </visual>
         <collision>
             <geometry>
-                <box size="0.6200000 0.585000 0.235000" />
+                <box size="0.62 0.585 0.235" />
             </geometry>
         </collision>
@@ -43,42 +31,9 @@
         </gazebo>
     </link>
-    <!-- Inertial link -->
-    <link name="inertial_link">
-        <inertial>
-            <mass value="132.3898489950015" />
-            <origin xyz="0 0 0.5" />
-            <inertia ixx="0.185196122711036"
-                     ixy="4.30144213829512E-08"
-                     ixz="5.81037523686401E-08"
-                     iyy="0.364893736238929"
-                     iyz="-0.000386720198091934"
-                     izz="0.223868521722778" />
-        </inertial>
-        <gazebo/>
-    </link>
-    <!-- Inertial joint -->
-    <joint name="inertial_joint" type="fixed">
-        <origin xyz="0 0 0" rpy="0 0 0" />
-        <parent link="base_link" />
-        <child link="inertial_link" />
-    </joint>
-    <!-- Scout wheel macros -->
-    <!-- wheel labeled from 0 to 3, counter-clockwise, starting from front right wheel -->
-    <!-- motor 1 and 2 (left side) are mechanically installed in a reversed direction -->
-    <xacro:scout_mini_wheel_1 wheel_prefix="rear_right">
-        <origin xyz="${wheelbase / 2} ${-track / 2} ${wheel_vertical_offset}" rpy="0 1.57 0" />
-    </xacro:scout_mini_wheel_1>
-    <xacro:scout_mini_wheel_2 wheel_prefix="front_right">
-        <origin xyz="${wheelbase / 2} ${track / 2} ${wheel_vertical_offset}" rpy="0 1.57 0" />
-    </xacro:scout_mini_wheel_2>
-    <xacro:scout_mini_wheel_3 wheel_prefix="front_left">
-        <origin xyz="${-wheelbase / 2} ${track / 2} ${wheel_vertical_offset}" rpy="0 -1.57 0" />
-    </xacro:scout_mini_wheel_3>
-    <xacro:scout_mini_wheel_4 wheel_prefix="rear_left">
-        <origin xyz="${-wheelbase / 2} ${-track / 2} ${wheel_vertical_offset}" rpy="0 -1.57 0" />
-    </xacro:scout_mini_wheel_4>
+    <!-- Include Lidar sensor -->
+    <xacro:include filename="$(find scout_description)/urdf/lidar_sensor.xacro" />
     <!-- Additional definitions -->
     <xacro:include filename="$(arg urdf_extras)" />
-    <!-- Gazebo definitions  -->
+    <!-- Gazebo definitions -->
     <xacro:include filename="$(find scout_description)/urdf/scout_mini.gazebo" />
 </robot>

File: scout/scout_description/urdf/scout_mini_wheel_1.xacro (robot description, xacro)
@@ -24,50 +24,31 @@
 -->
 <robot xmlns:xacro="http://ros.org/wiki/xacro" name="scout_wheel">
-    <xacro:macro name="scout_mini_wheel_1" params="wheel_prefix *joint_pose">
-        <link name="${wheel_prefix}_wheel_link">
-            <!--<inertial>
-                <mass value="3" />
-                <origin
-                        xyz="0.162297526351145 -0.159063056237197 -0.159999952657767"
-                        rpy="0 0 0" />
-                        <inertia ixx="0.7171" ixy="0" ixz="0" iyy="0.1361" iyz="0" izz="0.7171" />
-                   </inertial>
-            <visual>
-                <origin xyz="0 0 0" rpy="0 0 0" />
-                <geometry>
-                    <mesh filename="package://scout_description/meshes/wheel.dae" />
-                </geometry>
-            </visual>-->
-            <inertial>
-                <mass value="3" />
-                <origin xyz="0 0 0" />
-                <inertia ixx="0.7171" ixy="0" ixz="0" iyy="0.7171" iyz="0" izz="0.1361" />
-                <!--<inertia ixx="0" ixy="0" ixz="0" iyy="0" iyz="0" izz="0" />-->
-            </inertial>
-            <visual>
-                <origin xyz="0 0 0" rpy="0 0 0" />
-                <geometry>
-                    <mesh filename="package://scout_description/meshes/wheel.dae" />
-                </geometry>
-            </visual>
-            <collision>
-              <origin
-                xyz="0 0 0"
-                rpy="0 0 0" />
-              <geometry>
-                <mesh
-                  filename="package://scout_description/meshes/wheel.dae" />
-              </geometry>
-            </collision>
-        </link>
-        <joint name="${wheel_prefix}_wheel" type="continuous">
-            <!--<origin
-                  xyz="0.14547 0.20835 -0.07424"
-                  rpy="0 1.57 0" />-->
-            <parent link="base_link"/>
-            <child link="${wheel_prefix}_wheel_link"/>
-            <xacro:insert_block name="joint_pose"/>
-            <axis xyz="0 0 -1" rpy="0 0 0" />
-        </joint>
-    </xacro:macro>
+  <xacro:macro name="scout_mini_wheel_1" params="wheel_prefix">
+    <link name="${wheel_prefix}_wheel_link">
+        <inertial>
+            <mass value="3" />
+            <origin xyz="0 0 0" />
+            <inertia ixx="0.7171" ixy="0" ixz="0" iyy="0.7171" iyz="0" izz="0.1361" />
+        </inertial>
+        <visual>
+            <origin xyz="0 0 0" rpy="0 0 0" />
+            <geometry>
+                <mesh filename="package://scout_description/meshes/wheel.dae" scale="0.1 0.1 0.1" />
+            </geometry>
+            <material name="Gazebo/Red"/>
+        </visual>
+        <collision>
+            <origin xyz="0 0 0" rpy="0 0 0" />
+            <geometry>
+                <cylinder radius="0.08" length="0.05" />
+            </geometry>
+        </collision>
+    </link>
+    <joint name="${wheel_prefix}_wheel" type="continuous">
+        <parent link="base_link"/>
+        <child link="${wheel_prefix}_wheel_link"/>
+        <origin xyz="0.14547 0.20835 -0.07424" rpy="0 1.57 0" />
+        <axis xyz="0 0 -1" />
+    </joint>
+  </xacro:macro>
 </robot>

File: scout/scout_description/urdf/scout_mini_wheel_2.xacro (robot description, xacro)
@@ -24,50 +24,36 @@
 -->
 <robot xmlns:xacro="http://ros.org/wiki/xacro" name="scout_wheel">
-    <xacro:macro name="scout_mini_wheel_2" params="wheel_prefix *joint_pose">
-        <link name="${wheel_prefix}_wheel_link">
-            <!--<inertial>
+  <xacro:macro name="scout_mini_wheel_2" params="wheel_prefix">
+    <link name="${wheel_prefix}_wheel_link">
+        <inertial>
             <mass value="3" />
-                <origin
-                        xyz="0.162297526351148 0.159063056237198 -0.160000047342231"
-                        rpy="0 0 0" />
-                        <inertia ixx="0.7171" ixy="0" ixz="0" iyy="0.1361" iyz="0" izz="0.7171" />
-            </inertial>
-            <visual>
-                <origin xyz="0 0 0" rpy="0 0 0" />
-                <geometry>
-                    <mesh filename="package://scout_description/meshes/wheel.dae" />
-                </geometry>
-            </visual>-->
-            <inertial>
-                <mass value="3" />
-                <origin xyz="0 0 0" />
-                <inertia ixx="0.7171" ixy="0" ixz="0" iyy="0.7171" iyz="0" izz="0.1361" />
-                <!--<inertia ixx="0" ixy="0" ixz="0" iyy="0" iyz="0" izz="0" />-->
-            </inertial>
-            <visual>
-                <origin xyz="0 0 0" rpy="0 0 0" />
-                <geometry>
-                    <mesh filename="package://scout_description/meshes/wheel.dae" />
-                </geometry>
-            </visual>
-            <collision>
-              <origin
-                xyz="0 0 0"
-                rpy="0 0 0" />
-              <geometry>
-                <mesh
-                  filename="package://scout_description/meshes/wheel.dae" />
-              </geometry>
-            </collision>
-        </link>
-        <joint name="${wheel_prefix}_wheel" type="continuous">
-            <!--<origin
-                  xyz="-0.17453 0.20835 -0.07424"
-                  rpy="0 -1.57 0" />-->
-            <parent link="base_link"/>
-            <child link="${wheel_prefix}_wheel_link"/>
-            <xacro:insert_block name="joint_pose"/>
-            <axis xyz="0 0 -1" rpy="0 0 0" />
-        </joint>
-    </xacro:macro>
+            <origin xyz="0 0 0" />
+            <inertia ixx="0.7171" ixy="0" ixz="0" iyy="0.7171" iyz="0" izz="0.1361" />
+        </inertial>
+        <visual>
+            <origin xyz="0 0 0" rpy="0 0 0" />
+            <geometry>
+                <mesh filename="package://scout_description/meshes/wheel.dae" />
+            </geometry>
+            <material name="wheel_material">
+              <color rgba="1.0 0.0 0.0 1.0"/>
+            </material>
+        </visual>
+        <collision>
+            <origin xyz="0 0 0" rpy="0 0 0" />
+            <geometry>
+                <mesh filename="package://scout_description/meshes/wheel.dae" />
+            </geometry>
+        </collision>
+        <gazebo>
+          <material>Gazebo/Red</material>
+        </gazebo>
+    </link>
+    <joint name="${wheel_prefix}_wheel" type="continuous">
+        <parent link="base_link"/>
+        <child link="${wheel_prefix}_wheel_link"/>
+        <origin xyz="-0.17453 0.20835 -0.07424" rpy="0 -1.57 0" />
+        <axis xyz="0 0 -1" />
+    </joint>
+  </xacro:macro>
 </robot>

File: scout/scout_description/urdf/scout_mini_wheel_3.xacro (robot description, xacro)
@@ -24,50 +24,36 @@
 -->
 <robot xmlns:xacro="http://ros.org/wiki/xacro" name="scout_wheel">
-    <xacro:macro name="scout_mini_wheel_3" params="wheel_prefix *joint_pose">
-        <link name="${wheel_prefix}_wheel_link">
-            <!--<inertial>
+  <xacro:macro name="scout_mini_wheel_3" params="wheel_prefix">
+    <link name="${wheel_prefix}_wheel_link">
+        <inertial>
             <mass value="3" />
-                <origin
-                        xyz="-0.235088020493741 -0.0575697183039213 -0.16000004734223"
-                        rpy="0 0 0" />
-                        <inertia ixx="0.7171" ixy="0" ixz="0" iyy="0.1361" iyz="0" izz="0.7171" />
-            </inertial>
-            <visual>
-                <origin xyz="0 0 0" rpy="0 0 0" />
-                <geometry>
-                    <mesh filename="package://scout_description/meshes/wheel.dae" />
-                </geometry>
-            </visual>-->
-            <inertial>
-                <mass value="3" />
-                <origin xyz="0 0 0" />
-                <inertia ixx="0.7171" ixy="0" ixz="0" iyy="0.7171" iyz="0" izz="0.1361" />
-                <!--<inertia ixx="0" ixy="0" ixz="0" iyy="0" iyz="0" izz="0" />-->
-            </inertial>
-            <visual>
-                <origin xyz="0 0 0" rpy="0 0 0" />
-                <geometry>
-                    <mesh filename="package://scout_description/meshes/wheel.dae" />
-                </geometry>
-            </visual>
-            <collision>
-              <origin
-                xyz="0 0 0"
-                rpy="0 0 0" />
-              <geometry>
-                <mesh
-                  filename="package://scout_description/meshes/wheel.dae" />
-              </geometry>
-            </collision>
-        </link>
-        <joint name="${wheel_prefix}_wheel" type="continuous">
-            <!--<origin
-                  xyz="-0.17453 -0.24424 -0.07424"
-                  rpy="0 -1.57 0" />-->
-            <parent link="base_link"/>
-            <child link="${wheel_prefix}_wheel_link"/>
-            <xacro:insert_block name="joint_pose"/>
-            <axis xyz="0 0 -1" rpy="0 0 0" />
-        </joint>
-    </xacro:macro>
+            <origin xyz="0 0 0" />
+            <inertia ixx="0.7171" ixy="0" ixz="0" iyy="0.7171" iyz="0" izz="0.1361" />
+        </inertial>
+        <visual>
+            <origin xyz="0 0 0" rpy="0 0 0" />
+            <geometry>
+                <mesh filename="package://scout_description/meshes/wheel.dae" />
+            </geometry>
+            <material name="wheel_material">
+              <color rgba="1.0 0.0 0.0 1.0"/>
+            </material>
+        </visual>
+        <collision>
+            <origin xyz="0 0 0" rpy="0 0 0" />
+            <geometry>
+                <mesh filename="package://scout_description/meshes/wheel.dae" />
+            </geometry>
+        </collision>
+        <gazebo>
+          <material>Gazebo/Red</material>
+        </gazebo>
+    </link>
+    <joint name="${wheel_prefix}_wheel" type="continuous">
+        <parent link="base_link"/>
+        <child link="${wheel_prefix}_wheel_link"/>
+        <origin xyz="-0.17453 -0.24424 -0.07424" rpy="0 -1.57 0" />
+        <axis xyz="0 0 -1" />
+    </joint>
+  </xacro:macro>
 </robot>

File: scout/scout_description/urdf/scout_mini_wheel_4.xacro (robot description, xacro)
@@ -24,12 +24,10 @@
 -->
 <robot xmlns:xacro="http://ros.org/wiki/xacro" name="scout_wheel">
-    <xacro:macro name="scout_mini_wheel_4" params="wheel_prefix *joint_pose">
-        <link name="${wheel_prefix}_wheel_link">
-        <!--<inertial>
-        <mass value="3" />
-            <origin
-                    xyz="0.235244832119832 -0.0585653794466942 -0.206994929144493"
-                    rpy="0 0 0" />
-                    <inertia ixx="0.7171" ixy="0" ixz="0" iyy="0.1361" iyz="0" izz="0.7171" />
+  <xacro:macro name="scout_mini_wheel_4" params="wheel_prefix">
+    <link name="${wheel_prefix}_wheel_link">
+        <inertial>
+            <mass value="3" />
+            <origin xyz="0 0 0" />
+            <inertia ixx="0.7171" ixy="0" ixz="0" iyy="0.7171" iyz="0" izz="0.1361" />
         </inertial>
         <visual>
@@ -38,36 +36,24 @@
                 <mesh filename="package://scout_description/meshes/wheel.dae" />
             </geometry>
-        </visual>-->
-        <inertial>
-            <mass value="3" />
-            <origin xyz="0 0 0" />
-            <inertia ixx="0.7171" ixy="0" ixz="0" iyy="0.7171" iyz="0" izz="0.1361" />
-            <!--<inertia ixx="0" ixy="0" ixz="0" iyy="0" iyz="0" izz="0" />-->
-        </inertial>
-        <visual>
+            <material name="wheel_material">
+              <color rgba="1.0 0.0 0.0 1.0"/>
+            </material>
+        </visual>
+        <collision>
             <origin xyz="0 0 0" rpy="0 0 0" />
             <geometry>
                 <mesh filename="package://scout_description/meshes/wheel.dae" />
             </geometry>
-        </visual>
-            <collision>
-              <origin
-                xyz="0 0 0"
-                rpy="0 0 0" />
-              <geometry>
-                <mesh
-                  filename="package://scout_description/meshes/wheel.dae" />
-              </geometry>
-            </collision>
-        </link>
-        <joint name="${wheel_prefix}_wheel" type="continuous">
-            <!--<origin
-                  xyz="0.19247 -0.24486 -0.073441"
-                  rpy="-0 1.57 0" />-->
-            <parent link="base_link"/>
-            <child link="${wheel_prefix}_wheel_link"/>
-            <xacro:insert_block name="joint_pose"/>
-            <axis xyz="0 0 -1" rpy="0 0 0" />
-        </joint>
-    </xacro:macro>
+        </collision>
+        <gazebo>
+          <material>Gazebo/Red</material>
+        </gazebo>
+    </link>
+    <joint name="${wheel_prefix}_wheel" type="continuous">
+        <parent link="base_link"/>
+        <child link="${wheel_prefix}_wheel_link"/>
+        <origin xyz="0.19247 -0.24486 -0.073441" rpy="0 1.57 0" />
+        <axis xyz="0 0 -1" />
+    </joint>
+  </xacro:macro>
 </robot>
