Commit message: Fix lidar and wheel visibility issues

File: scout/scout_description/urdf/lidar_sensor.xacro (robot description, xacro)
@@ -24,5 +24,5 @@
   <!-- Joint to Base Link -->
   <joint name="lidar_joint" type="fixed">
-    <origin xyz="0 0 0.3" rpy="0 0 0" />
+    <origin xyz="0 0 0.2" rpy="0 0 0" />
     <parent link="base_link" />
     <child link="lidar_link" />

File: scout/scout_description/urdf/scout_mini.xacro (robot description, xacro)
@@ -1,39 +1,136 @@
-<?xml version="1.0"?>
-<robot name="scout_mini"
-       xmlns:xacro="http://ros.org/wiki/xacro">
-    <xacro:arg name="robot_namespace" default="/" />
-    <xacro:arg name="urdf_extras" default="$(find scout_description)/urdf/empty.urdf" />
-    <!-- Include wheel definitions -->
-    <xacro:include filename="$(find scout_description)/urdf/scout_mini_wheel_1.xacro" />
-    <xacro:include filename="$(find scout_description)/urdf/scout_mini_wheel_2.xacro" />
-    <xacro:include filename="$(find scout_description)/urdf/scout_mini_wheel_3.xacro" />
-    <xacro:include filename="$(find scout_description)/urdf/scout_mini_wheel_4.xacro" />
-    <!-- Base link -->
-    <link name="base_link">
-        <inertial>
-            <mass value="10" />
-            <origin xyz="0 0 0.5" />
-            <inertia ixx="0.1" ixy="0.0" ixz="0.0" iyy="0.1" iyz="0.0" izz="0.1" />
-        </inertial>
-        <visual>
-            <origin xyz="0.015 0.023 0" rpy="0 0 0"/>
-            <geometry>
-                <mesh filename="package://scout_description/meshes/scout_mini_base_link.STL" scale="1 1 1" />
-            </geometry>
-        </visual>
-        <collision>
-            <geometry>
-                <box size="0.62 0.585 0.235" />
-            </geometry>
-        </collision>
-        <gazebo>
-            <material>Gazebo/Blue</material>
-        </gazebo>
-    </link>
-    <!-- Include Lidar sensor -->
-    <xacro:include filename="$(find scout_description)/urdf/lidar_sensor.xacro" />
-    <!-- Additional definitions -->
-    <xacro:include filename="$(arg urdf_extras)" />
-    <!-- Gazebo definitions -->
-    <xacro:include filename="$(find scout_description)/urdf/scout_mini.gazebo" />
+<?xml version="1.0" ?>
+<robot xmlns:xacro="http://ros.org/wiki/xacro" name="scout_mini">
+  <!-- Base link -->
+  <link name="base_link">
+    <inertial>
+      <mass value="10"/>
+      <origin xyz="0 0 0.5"/>
+      <inertia ixx="0.1" ixy="0.0" ixz="0.0" iyy="0.1" iyz="0.0" izz="0.1"/>
+    </inertial>
+    <visual>
+      <origin rpy="0 0 0" xyz="0.015 0.023 0"/>
+      <geometry>
+        <mesh filename="package://scout_description/meshes/scout_mini_base_link.STL" scale="1 1 1"/>
+      </geometry>
+    </visual>
+    <collision>
+      <geometry>
+        <box size="0.62 0.585 0.235"/>
+      </geometry>
+    </collision>
+    <gazebo>
+      <material>Gazebo/Blue</material>
+    </gazebo>
+  </link>
+  <!-- Wheel links and joints -->
+  <link name="rear_right_wheel_link">
+    <inertial>
+      <mass value="3"/>
+      <origin xyz="0 0 0"/>
+      <inertia ixx="0.7171" ixy="0" ixz="0" iyy="0.7171" iyz="0" izz="0.1361"/>
+    </inertial>
+    <visual>
+      <origin rpy="0 0 0" xyz="0 0 0"/>
+      <geometry>
+        <mesh filename="package://scout_description/meshes/wheel.dae" scale="0.1 0.1 0.1"/>
+      </geometry>
+      <material name="Gazebo/Red"/>
+    </visual>
+    <collision>
+      <geometry>
+        <cylinder length="0.05" radius="0.08"/>
+      </geometry>
+    </collision>
+  </link>
+  <joint name="rear_right_wheel" type="continuous">
+    <parent link="base_link"/>
+    <child link="rear_right_wheel_link"/>
+    <origin rpy="0 1.57 0" xyz="0.14547 0.20835 -0.07424"/>
+    <axis xyz="0 0 -1"/>
+  </joint>
+  <link name="front_right_wheel_link">
+    <inertial>
+      <mass value="3"/>
+      <origin xyz="0 0 0"/>
+      <inertia ixx="0.7171" ixy="0" ixz="0" iyy="0.7171" iyz="0" izz="0.1361"/>
+    </inertial>
+    <visual>
+      <origin rpy="0 0 0" xyz="0 0 0"/>
+      <geometry>
+        <mesh filename="package://scout_description/meshes/wheel.dae"/>
+      </geometry>
+      <material name="Gazebo/Blue"/>
+    </visual>
+    <collision>
+      <geometry>
+        <mesh filename="package://scout_description/meshes/wheel.dae"/>
+      </geometry>
+    </collision>
+    <gazebo>
+      <material>Gazebo/Blue</material>
+    </gazebo>
+  </link>
+  <joint name="front_right_wheel" type="continuous">
+    <parent link="base_link"/>
+    <child link="front_right_wheel_link"/>
+    <origin rpy="0 -1.57 0" xyz="-0.17453 0.20835 -0.07424"/>
+    <axis xyz="0 0 -1"/>
+  </joint>
+  <link name="front_left_wheel_link">
+    <inertial>
+      <mass value="3"/>
+      <origin xyz="0 0 0"/>
+      <inertia ixx="0.7171" ixy="0" ixz="0" iyy="0.7171" iyz="0" izz="0.1361"/>
+    </inertial>
+    <visual>
+      <origin rpy="0 0 0" xyz="0 0 0"/>
+      <geometry>
+        <mesh filename="package://scout_description/meshes/wheel.dae"/>
+      </geometry>
+      <material name="Gazebo/Green"/>
+    </visual>
+    <collision>
+      <geometry>
+        <mesh filename="package://scout_description/meshes/wheel.dae"/>
+      </geometry>
+    </collision>
+    <gazebo>
+      <material>Gazebo/Green</material>
+    </gazebo>
+  </link>
+  <joint name="front_left_wheel" type="continuous">
+    <parent link="base_link"/>
+    <child link="front_left_wheel_link"/>
+    <origin rpy="0 -1.57 0" xyz="-0.17453 -0.24424 -0.07424"/>
+    <axis xyz="0 0 -1"/>
+  </joint>
+  <link name="rear_left_wheel_link">
+    <inertial>
+      <mass value="3"/>
+      <origin xyz="0 0 0"/>
+      <inertia ixx="0.7171" ixy="0" ixz="0" iyy="0.7171" iyz="0" izz="0.1361"/>
+    </inertial>
+    <visual>
+      <origin rpy="0 0 0" xyz="0 0 0"/>
+      <geometry>
+        <mesh filename="package://scout_description/meshes/wheel.dae"/>
+      </geometry>
+      <material name="Gazebo/Yellow"/>
+    </visual>
+    <collision>
+      <geometry>
+        <mesh filename="package://scout_description/meshes/wheel.dae"/>
+      </geometry>
+    </collision>
+    <gazebo>
+      <material>Gazebo/Yellow</material>
+    </gazebo>
+  </link>
+  <joint name="rear_left_wheel" type="continuous">
+    <parent link="base_link"/>
+    <child link="rear_left_wheel_link"/>
+    <origin rpy="0 1.57 0" xyz="0.19247 -0.24486 -0.073441"/>
+    <axis xyz="0 0 -1"/>
+  </joint>
+  <xacro:include filename="$(find scout_description)/urdf/lidar_sensor.xacro" />
 </robot>
